File: hardware/kicad/CatMouse.kicad_pcb (KiCad board)
At the start: 2 copper layers, 70 x 80 mm, 34 parts, among them J1 Power, J10 USB_B_Micro, J11 Motor1, J12 Motor2, J13 Motor3, J14 Motor4, J15 I2C0, J16 I2C0, J17 I2C1, J18 I2C1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

Commit message: board v0.4
Parts:
- removed J17, J18: I2C1, Connector_PinHeader_2.54mm:PinHeader_1x04_P2.54mm_Vertical
- removed R4, R5: 4.7k, Resistor_SMD:R_0805_2012Metric_Pad1.20x1.40mm_HandSolder
- added J19: Lidar, CatMouse:JST_ZH_B4B-ZR_1x04_P1.50mm_Vertical, F.Cu at (179.8, 124.0)
Connections:
- U2 pad 38: /SDA1 -> /LD_PWM
- U2 pad 39: /SCL1 -> /LD_RX
Routing:
- net /SCL1: track 103.9 -> 0.00 mm, vias 2 -> 0
- net /SDA1: track 96.7 -> 0.00 mm, vias 2 -> 0
- net /LD_RX: track 0.00 -> 81.8 mm, vias 0 -> 2
- net /LD_PWM: track 0.00 -> 81.3 mm, vias 0 -> 2
- net VCC: track 68.0 -> 126.1 mm, vias 4 -> 5
- net +3V3: track 426.7 -> 408.0 mm
Other:
- board text added: "PWM"
- board text added: "TX"
- board text added: "VCC"
