File: hardware/kicad/CatMouse.kicad_pcb (KiCad board)
At the start: 2 copper layers, 70 x 80 mm, 31 parts, among them J1 Power, J10 USB_B_Micro, J11 Motor1, J12 Motor2, J13 Motor3, J14 Motor4, J15 I2C0, J16 I2C0, J19 Lidar, J2 VCC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

Commit message: board 0.5 & fusion360 & stl files
Parts:
- added Q1: SL3007-TP, Package_TO_SOT_SMD:SOT-23, F.Cu at (176.9, 129.6)
- added R4: 10k, Resistor_SMD:R_0805_2012Metric_Pad1.20x1.40mm_HandSolder, F.Cu at (172.2, 128.7)
- J9: footprint Connector_PinHeader_2.54mm:PinHeader_1x06_P2.54mm_Vertical -> Connector_PinHeader_2.54mm:PinHeader_1x08_P2.54mm_Vertical
Connections:
- J19 pad 1: VCC -> /LD_PWR
- J19 pad 3: /LD_PWM -> GND
- J9 pad 3: /IO39 -> /IO48
- J9 pad 4: /IO40 -> /IO45
- J9 pad 5: /IO41 -> /IO39
- J9 pad 6: /IO42 -> /IO40
- U2 pad 25: unconnected-(U2-GPIO48/SPICLK_N/SUBSPICLK_N_DIFF-Pad25) -> /IO48
- U2 pad 26: unconnected-(U2-GPIO45-Pad26) -> /IO45
- U2 pad 38: /LD_PWM -> /~{LD_EN}
Routing:
- net /~{LD_EN}: track 0.00 -> 95.5 mm, vias 0 -> 2
- net /LD_PWM: track 81.3 -> 0.00 mm, vias 2 -> 0
- net /IO48: track 0.00 -> 36.6 mm
- net /IO45: track 0.00 -> 32.6 mm
- net /LD_PWR: track 0.00 -> 6.49 mm
- net /IO39: track 38.4 -> 33.3 mm
- net /IO41: track 35.0 -> 29.9 mm
- net /IO40: track 36.7 -> 31.7 mm
- net VCC: track 126.1 -> 121.1 mm
- net /IO42: track 33.3 -> 28.4 mm
- net /SCL0: track 75.1 -> 72.4 mm
- net /SDA0: track 68.4 -> 66.1 mm
- net +3V3: track 408.0 -> 407.0 mm
- net /M3_ENC1: track 39.8 -> 39.0 mm
Other:
- board text added: "IO45"
- board text added: "IO48"
- board text added: "V3V"
