File: hardware/kicad/CatMouse.kicad_sch (KiCad schematic)
At the start: 34 parts, among them J1 Power, J10 USB_B_Micro, J11 Motor1, J12 Motor2, J13 Motor3, J14 Motor4, J15 I2C0, J16 I2C0, J17 I2C1, J18 I2C1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

Commit message: board v0.4
Parts:
- removed J17, J18: I2C1, Connector_PinHeader_2.54mm:PinHeader_1x04_P2.54mm_Vertical, symbol Connector_Generic:Conn_01x04
- removed R4, R5: 4.7k, Resistor_SMD:R_0805_2012Metric_Pad1.20x1.40mm_HandSolder, symbol Device:R
- added J19: Lidar, CatMouse:JST_ZH_B4B-ZR_1x04_P1.50mm_Vertical, symbol Connector_Generic:Conn_01x04
Connections:
- net GND: now also J19.2 (Pin_2)
- net VCC: now also J19.1 (Pin_1)
- net SCL1 renamed LD_RX
- net LD_RX: now also J19.4 (Pin_4)
- net SDA1 renamed LD_PWM
- net LD_PWM: now also J19.3 (Pin_3)
Other:
- moved on the sheet: C1, C4, J10, J11, J15, J16, J4, J5, J6, J7, J8, J9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

Commit message: board 0.5 & fusion360 & stl files
Parts:
- added Q1: SL3007-TP, Package_TO_SOT_SMD:SOT-23, symbol Transistor_FET:Si2371EDS
- added R4: 10k, Resistor_SMD:R_0805_2012Metric_Pad1.20x1.40mm_HandSolder, symbol Device:R
- J9: footprint Connector_PinHeader_2.54mm:PinHeader_1x06_P2.54mm_Vertical -> Connector_PinHeader_2.54mm:PinHeader_1x08_P2.54mm_Vertical; symbol Connector_Generic:Conn_01x06 -> Connector_Generic:Conn_01x08
Connections:
- net GND: now also J19.3 (Pin_3)
- net IO39: now also J9.5 (Pin_5); no longer J9.3 (Pin_3)
- net IO40: now also J9.6 (Pin_6); no longer J9.4 (Pin_4)
- net IO41: now also J9.7 (Pin_7); no longer J9.5 (Pin_5)
- net IO42: now also J9.8 (Pin_8); no longer J9.6 (Pin_6)
- net VCC: now also Q1.2 (S), R4.1; no longer J19.1 (Pin_1)
- net IO48: now reaches U2.25 (GPIO48/SPICLK_N/SUBSPICLK_N_DIFF)
- net IO48: now also J9.3 (Pin_3)
- net IO45: now reaches U2.26 (GPIO45)
- net IO45: now also J9.4 (Pin_4)
- net LD_PWM renamed ~{LD_EN}
- net ~{LD_EN}: now also Q1.1 (G), R4.2; no longer J19.3 (Pin_3)
- new net LD_PWR: J19.1 (Pin_1), Q1.3 (D)
- no-connect marks 12 -> 10
Other:
- moved on the sheet: J19
